File: powerOutageLogger.brd (EAGLE design)
At the start: 99.1 x 74.9 mm, 32 parts, among them J1 2.1MMJACKTHM, U1 ATmega328P, U2 78L05, Y1 16MHz

Commit message: v1.1
Parts:
- added C10: 100nF, _jc:C025-025X050
- added U$2: (no value), ohw-logo:OSHW_8X200_NOTEXT
- C7: value 27pF -> 100nF
- C9: value 100nF -> 27pF
- S1, S2: device _jc:B3F-10XXOCT -> _jc:B3F-312X
- S3: value DOWN -> DN; device _jc:B3F-10XXOCT -> _jc:B3F-312X
- moved J1 101.1 mm to (95.2, 12.7), turned to 270 degrees
- moved D1 90.7 mm to (85.1, 3.81), turned to 0 degrees
- moved C2 78.2 mm to (80.0, 7.62), turned to 180 degrees
- moved C1 74.5 mm to (80.0, 17.8), turned to 180 degrees
- moved U2 72.8 mm to (80.0, 11.4), turned to 0 degrees
- moved JP1 68.8 mm to (72.4, 3.81), turned to 90 degrees
- moved D3 66.1 mm to (78.7, 71.1)
- moved S1 66.1 mm to (21.6, 71.1)
- moved S3 66.1 mm to (59.7, 71.1)
- moved S2 66.0 mm to (40.6, 71.1)
- moved S4 65.4 mm to (64.8, 25.4), turned to 0 degrees
- moved C3 62.3 mm to (73.4, 17.8), turned to 0 degrees
- moved C4 61.4 mm to (73.7, 13.5), turned to 0 degrees
- moved PCB1 56.4 mm to (35.6, 15.2), turned to 90 degrees
- moved JP2 54.6 mm to (55.9, 10.2), turned to 90 degrees
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Connections:
- removed net PD4: JP2.3, U1.6
- removed net PD5: S2.1, S2.2, U1.11
- removed net PD6: S1.1, S1.2, U1.12
- net /RESET: now also C10.1; no longer C9.1
- net GND: now also C9.2, S1.1, S2.1, S3.1; no longer S1.3, S1.4, S2.3, S2.4, S3.3, S3.4
- net MOSI: now also S1.2
- net N$9: now also C7.1; no longer C5.1
- net PC3: now also PCB2.6; no longer PCB2.4
- net PD2: now also PCB2.4; no longer PCB2.6
- net PD3: now also JP2.3
- net PD7: no longer S3.1
- net RST: now also C10.2; no longer C9.2
- net SS: now also S2.2
- net VCC: now also C5.1
- net XTAL1: now also C9.1; no longer C8.1
- net XTAL2: now also C8.1; no longer C7.1
Routing:
- net /RESET: track 155.6 -> 81.8 mm
- net PD6: track 70.5 -> 0.00 mm
- net PD5: track 58.9 -> 0.00 mm
- net MOSI: track 43.8 -> 101.8 mm
- net N$3: track 11.3 -> 67.8 mm
- net PD4: track 42.9 -> 0.00 mm
- net SS: track 0.00 -> 41.7 mm
- net PD3: track 0.00 -> 33.9 mm
- net VCC: track 192.7 -> 219.8 mm
- net PC2: track 30.0 -> 50.9 mm
- net SCL: track 46.3 -> 31.6 mm
- net PB1: track 31.5 -> 18.5 mm
- net PD7: track 23.3 -> 32.2 mm
- net N$5: track 27.9 -> 20.6 mm
- net SDA: track 38.3 -> 32.4 mm
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Other:
- board text added: "12345"
- board text added: "CC BY-SA jc 0912 v1.1"
- board text added: "http://github.com/JChristensen"
- board text removed: "CC BY-SA jc 0912 v1.0"

Commit message: v1.1
Parts:
- added R5: 0, _jc:0204/6
- moved R3 2.84 mm to (69.8, 57.7)
- moved U$1 1.27 mm to (1.27, 64.8)
Connections:
- new net N$6: PCB2.15, R5.2
- net PB1: now also R5.1; no longer PCB2.15
Routing:
- net N$6: track 0.00 -> 15.0 mm
- net PB1: track 18.5 -> 4.34 mm
- net PB0: track 11.2 -> 13.5 mm
- net N$4: track 15.9 -> 13.6 mm
- net SS: track 41.7 -> 40.2 mm
- net PD3: track 33.9 -> 35.2 mm
- net MOSI: track 101.8 -> 101.0 mm

Commit message: Version 1.1 Added ReadMe.txt Added schematic.png
Parts:
- added R6: 4.7K, _jc:0204/6
- added TB1: Ext Sensor, _jc:OST-TB-3-3.5MM
- added U3: DS18B20, _jc:TO92-OVAL
- moved JP4 43.9 mm to (54.6, 6.35), turned to 0 degrees
- moved JP2 29.0 mm to (27.9, 17.8), turned to 0 degrees
- moved C10 15.3 mm to (26.7, 53.3), turned to 90 degrees
- moved S4 8.52 mm to (57.1, 21.6)
- moved C9 8.29 mm to (56.1, 33.0), turned to 0 degrees
- moved C8 4.44 mm to (50.5, 33.0), turned to 180 degrees
- moved Y1 2.59 mm to (53.3, 37.3)
- moved C5 1.48 mm to (44.5, 38.1)
- moved J1 1.27 mm to (95.2, 11.4)
- moved R3 1.27 mm to (69.8, 58.9)
- moved R5 1.27 mm to (66.0, 58.9)
Connections:
- new net PD6: R6.2, TB1.P$2, U1.12, U3.2
- net GND: now also TB1.P$3, U3.1
- net VCC: now also R6.1, TB1.P$1, U3.3
Routing:
- net PD6: track 0.00 -> 48.7 mm
- net VCC: track 219.8 -> 267.5 mm
- net RST: track 21.2 -> 12.4 mm
- net /RESET: track 81.8 -> 73.4 mm
- net PD3: track 35.2 -> 40.6 mm
- net MOSI: track 101.0 -> 105.7 mm
- net N$5: track 20.6 -> 16.7 mm
- net XTAL1: track 13.6 -> 11.1 mm
- net XTAL2: track 12.5 -> 11.1 mm
- net N$1: track 30.1 -> 28.7 mm
- net N$4: track 13.6 -> 12.3 mm
- net PB1: track 4.34 -> 5.61 mm
- net PB0: track 13.5 -> 14.8 mm
Other:
- board text added: "Clock"
- board text added: "FTDI"
- board text added: "GND"
- board text added: "Real-Time"
- board text removed: "Hack Me"
- board text removed: "Real-Time Clock"

Commit message: Minor trace tweaks.
Parts:
- moved R6 7.28 mm to (71.9, 25.9)
- moved U3 1.27 mm to (67.3, 25.4)
- moved D1 0.92 mm to (84.3, 4.32)
Routing:
- net N$3: track 67.8 -> 54.7 mm
- net VCC: track 267.5 -> 262.0 mm
- net PD6: track 48.7 -> 50.5 mm
- net PD3: track 40.6 -> 39.3 mm
- net N$1: track 28.7 -> 27.5 mm
Other:
- board text added: "5VDC regulated input."
- board text added: "Input power jumper (PWR SEL):"
- board text added: "Use DIRECT position only for"
- board text added: "Use REG position for 7-12VDC input."
